File: test_bench_pico/test_bench_pico.kicad_pcb (KiCad board)
At the start: 2 copper layers, 140 x 120 mm, 68 parts, among them J1 12V_IN_20A, J2 MOTOR_20A, J3 UPDI, J4 RS485_A_B_GND, J5 SENSOR1_12V_SIG_GND, J6 SENSOR2_12V_SIG_GND, J7 SENSOR3_12V_SIG_GND, J8 SENSOR4_12V_SIG_GND, Q1 CSD18540Q5B HS-A, Q2 CSD18540Q5B LS-A, Q3 CSD18540Q5B HS-B, Q4 CSD18540Q5B LS-B, U1 DRV8701ERGER, U2 ATtiny1616-MNR, U3 THVD1429DR, U4 LTV-817S, U5 LTV-817S, U6 LTV-817S, U7 LTV-817S

Commit message: Improve PCB routing and schematic workflows
Parts:
- moved CS1 94.8 mm to (122.0, 62.0)
- moved U4 79.9 mm to (106.0, 70.0)
- moved RP1 75.4 mm to (106.0, 65.0)
- moved U2 57.7 mm to (126.0, 62.0), turned to -90 degrees
- moved R7 55.0 mm to (130.0, 66.0)
- moved D3 49.4 mm to (130.0, 70.0), turned to 90 degrees
- moved R3 48.3 mm to (130.0, 62.0), turned to 90 degrees
- moved J4 46.4 mm to (116.0, 80.0), turned to 180 degrees
- moved R1 43.3 mm to (121.0, 58.0), turned to 90 degrees
- moved C9 40.8 mm to (138.0, 85.0), turned to -90 degrees
- moved C8 35.2 mm to (88.0, 112.0)
- moved C6 34.5 mm to (116.0, 56.0), turned to -90 degrees
- moved DS1 34.4 mm to (57.0, 132.0)
- moved R2 34.2 mm to (107.0, 56.0), turned to 180 degrees
- moved D2 29.1 mm to (123.0, 76.0), turned to -90 degrees
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Routing:
- net /VMOTOR: track 0.00 -> 381.6 mm
- net /5V_DVDD: track 0.00 -> 176.2 mm, vias 0 -> 3
- net /SENSOR2_N: track 0.00 -> 113.7 mm, vias 0 -> 3
- net /UPDI: track 0.00 -> 109.5 mm, vias 0 -> 3
- net /SENSOR1_LED_A: track 0.00 -> 106.7 mm, vias 0 -> 2
- net /RS485_B: track 0.00 -> 73.4 mm, vias 0 -> 1
- net /SENSOR4_N: track 0.00 -> 66.3 mm, vias 0 -> 2
- net /RS485_A: track 0.00 -> 58.7 mm, vias 0 -> 2
- net /DRIVER_SLEEP: track 0.00 -> 51.8 mm
- net /SENSOR3_LED_A: track 0.00 -> 43.8 mm, vias 0 -> 2
- net /SENSOR4_LED_A: track 0.00 -> 38.4 mm
- net /MOTOR_B: track 0.00 -> 36.2 mm
- net /CURRENT_SENSE: track 0.00 -> 34.2 mm
- net /DRIVER_FAULT: track 0.00 -> 29.7 mm, vias 0 -> 3
- net /GATE_LS_B: track 0.00 -> 29.6 mm
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